File: programs/DAC8822/pcb/DAC8822.kicad_pcb (KiCad board)
At the start: 2 copper layers, 102.1 x 44 mm, 17 parts, among them J1 TFT ST7735, U1 8BVG4, U2 8BVG4, U3 RP2350B-WeAct, U4 OPA2277, U5 OPA2277, U6 OPA2277, U7 OPA2277, U8 LM7805

Commit message: Add files via upload
Parts:
- added J2: Conn_01x04_Pin, Connector_PinHeader_1.00mm:PinHeader_1x04_P1.00mm_Vertical, F.Cu at (85.8, 91.9)
- added J3: Conn_01x04_Pin, Connector_PinHeader_1.00mm:PinHeader_1x04_P1.00mm_Vertical, F.Cu at (85.8, 105.6)
- added J4: Screw_Terminal_01x02, TerminalBlock:TerminalBlock_Xinya_XY308-2.54-2P_1x02_P2.54mm_Horizontal, F.Cu at (183.2, 75.4)
- added J5: Conn_01x04_Pin, Connector_PinHeader_1.00mm:PinHeader_1x04_P1.00mm_Vertical, F.Cu at (144.0, 124.4)
- added J6: Conn_01x04_Pin, Connector_PinHeader_1.00mm:PinHeader_1x04_P1.00mm_Vertical, F.Cu at (151.1, 124.3)
- moved C1 0.20 mm to (91.0, 89.6)
- moved C2 0.20 mm to (91.0, 96.3)
- moved C3 0.20 mm to (91.0, 103.6)
- moved C4 0.20 mm to (91.0, 110.1)
- moved U4 0.20 mm to (98.0, 89.8)
- moved U5 0.20 mm to (98.0, 96.3)
- moved U6 0.20 mm to (98.0, 103.6)
- moved U7 0.20 mm to (98.0, 110.1)
Connections:
- U2 pad 15: unconnected-(U2-R_{1}B-Pad15) -> Vref
- U2 pad 17: unconnected-(U2-R_{OFS}B-Pad17) -> Vref
- U2 pad 3: +10V -> Vref
- U2 pad 5: +10V -> Vref
- U3 pad 38: unconnected-(U3-GPIO32-Pad38) -> /Btn1
- U3 pad 39: unconnected-(U3-GPIO33-Pad39) -> /Btn2
- U3 pad 40: unconnected-(U3-GPIO34-Pad40) -> /Btn3
- U3 pad 41: unconnected-(U3-GPIO35-Pad41) -> /Btn4
- U3 pad 46: unconnected-(U3-GPIO40_ADC0-Pad46) -> /Pot1
- U3 pad 47: unconnected-(U3-GPIO41_ADC1-Pad47) -> /Pot2
- U3 pad 55: unconnected-(U3-3V3-Pad55) -> +3.3V
- U3 pad 56: unconnected-(U3-3V3-Pad56) -> +3.3V
- U9 pad 1: unconnected-(U9-VIN-Pad1) -> +BATT
Routing:
- net +12V: track 30.8 -> 150.6 mm, vias 0 -> 5
- net -12V: track 0.00 -> 111.0 mm, vias 0 -> 4
- net +5V: track 75.3 -> 158.4 mm
- net /Btn2: track 0.00 -> 45.5 mm
- net /Btn1: track 0.00 -> 43.6 mm
- net Vref: track 0.00 -> 41.7 mm, vias 0 -> 4
- net /Btn3: track 0.00 -> 39.2 mm
- net /Btn4: track 0.00 -> 35.6 mm
- net /Pot1: track 0.00 -> 28.2 mm
- net /Pot2: track 0.00 -> 24.5 mm
- net /Ch2: track 0.00 -> 24.4 mm
- net /Ch4: track 0.00 -> 23.7 mm
- net Net-(U1-I_{OUT}A): track 0.00 -> 23.1 mm, vias 0 -> 2
- net Net-(U2-I_{OUT}A): track 0.00 -> 22.4 mm, vias 0 -> 2
- net /Ch3: track 0.00 -> 21.9 mm
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Other:
- board size 102.1 x 44 mm -> 105 x 57.2 mm

Commit message: Add files via upload
Parts:
- added R1: 100, Resistor_SMD:R_0805_2012Metric, F.Cu at (96.0, 118.1)
- added R2: 3k, Resistor_SMD:R_0805_2012Metric, F.Cu at (96.0, 121.1)
- added R3: 1k, Resistor_SMD:R_0805_2012Metric, F.Cu at (96.0, 124.0)
- added U10: TL431LP, Package_TO_SOT_THT:TO-92_Inline, F.Cu at (100.2, 119.9)
- U9: value ~ -> Dual PSU
- moved J4 1.14 mm to (182.3, 76.1)
Connections:
- D1 pad 1: /VSYS -> /Vsys
- J1 pad 1: +5V -> /Vsys
- U3 pad 2: /VSYS -> /Vsys
Routing:
- net /Vsys: track 0.00 -> 98.0 mm
- net /VSYS: track 81.2 -> 0.00 mm
- net +5V: track 158.4 -> 131.5 mm
- net Vref: track 41.7 -> 65.0 mm
- net GND: track 19.1 -> 0.27 mm
- net Net-(U10-REF): track 0.00 -> 7.47 mm
- net +12V: track 150.6 -> 156.9 mm
- net +BATT: track 14.9 -> 13.8 mm
Other:
- board text added: "+"
- board text added: "-"
- board text added: "Batt"

Commit message: Add files via upload
Parts:
- J2, J3, J5, J6: footprint Connector_PinHeader_1.00mm:PinHeader_1x04_P1.00mm_Vertical -> Connector_PinHeader_1.27mm:PinHeader_1x04_P1.27mm_Vertical
- U9: value Dual PSU -> ~
Connections:
- R2 pad 1: Vref -> Net-(U10-REF)
- R2 pad 2: Net-(U10-REF) -> Vref
Routing:
- net GND: track 0.27 -> 13.2 mm, vias 0 -> 26
- net +12V: track 156.9 -> 161.8 mm
- net Net-(U10-REF): track 7.47 -> 10.6 mm
- net /~{CS}: track 41.1 -> 42.9 mm
- net /D1: track 32.3 -> 33.1 mm
- net /Ch2: track 24.4 -> 23.8 mm
- net /Ch4: track 23.7 -> 23.2 mm
- added copper zone on B.Cu, net GND
- added copper zone on F.Cu, net GND

Commit message: Add files via upload
Parts:
- moved R1 1.22 mm to (96.0, 116.9)
- moved R2 1.22 mm to (96.0, 119.8)
- moved R3 1.22 mm to (96.0, 122.8)
- moved U10 1.22 mm to (100.2, 118.7)
- moved J1 1.20 mm to (138.2, 100.9)
Routing:
- net GND: track 13.2 -> 31.7 mm, vias 26 -> 18
- net +5V: track 131.5 -> 125.1 mm
- net +3.3V: track 13.5 -> 18.9 mm
- net /U1: track 70.9 -> 76.2 mm
- net /D2: track 35.5 -> 39.8 mm, vias 0 -> 2
- net /~{RS}: track 81.3 -> 77.2 mm, vias 5 -> 4
- net /D5: track 28.9 -> 32.8 mm, vias 2 -> 4
- net /D15: track 67.4 -> 64.0 mm
- net /Pot1: track 28.3 -> 31.4 mm
- net /Btn1: track 43.6 -> 46.5 mm
- net /D3: track 26.8 -> 29.6 mm, vias 2 -> 4
- net /D8: track 35.8 -> 38.5 mm
- net /Vsys: track 98.0 -> 95.5 mm, vias 0 -> 1
- net /Btn3: track 39.4 -> 41.7 mm
- net /~{WR}: track 92.7 -> 94.9 mm
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Other:
- board size 105 x 57.2 mm -> 105 x 58 mm

Commit message: Add files via upload
Parts:
- added C10: 0.1uF, Capacitor_SMD:C_0805_2012Metric, B.Cu at (96.1, 96.6)
- added C11: 0.1uF, Capacitor_SMD:C_0805_2012Metric, B.Cu at (96.3, 104.2)
- added C12: 0.1uF, Capacitor_SMD:C_0805_2012Metric, B.Cu at (96.0, 108.9)
- added C7: 0.1uF, Capacitor_SMD:C_0805_2012Metric, B.Cu at (108.0, 114.8)
- added C8: 0.1uF, Capacitor_SMD:C_0805_2012Metric, B.Cu at (112.9, 81.7)
- added C9: 0.1uF, Capacitor_SMD:C_0805_2012Metric, B.Cu at (96.3, 90.2)
- moved J4 2.66 mm to (185.0, 76.2)
- moved D1 2.20 mm to (185.2, 108.5)
- moved C5 2.20 mm to (176.9, 117.0)
- moved C6 2.20 mm to (170.9, 117.0)
- moved U8 2.20 mm to (172.7, 111.5)
- moved U9 2.00 mm to (178.7, 93.1)
- moved J1 1.90 mm to (140.1, 101.0)
Connections:
- net Net-(U10-REF) renamed /Adj
Routing:
- net +3.3V: track 18.9 -> 55.4 mm, vias 0 -> 1
- net /Btn2: track 45.3 -> 22.2 mm, vias 0 -> 1
- net /Btn1: track 46.5 -> 24.1 mm, vias 0 -> 1
- net +5V: track 125.1 -> 144.8 mm, vias 2 -> 4
- net GND: track 31.7 -> 13.2 mm, vias 18 -> 19
- net /LED: track 5.61 -> 23.1 mm
- net /SCK: track 65.2 -> 49.8 mm, vias 1 -> 0
- net -12V: track 112.4 -> 126.7 mm
- net +12V: track 160.6 -> 173.8 mm
- net /Pot2: track 24.9 -> 37.4 mm, vias 0 -> 1
- net /Btn3: track 41.7 -> 29.9 mm, vias 0 -> 1
- net /U2: track 60.1 -> 48.4 mm, vias 2 -> 0
- net /Btn4: track 36.7 -> 27.5 mm, vias 0 -> 1
- net /D15: track 64.0 -> 72.5 mm, vias 4 -> 3
- net /SDA: track 72.3 -> 64.1 mm, vias 2 -> 0
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Other:
- board size 105 x 58 mm -> 107.7 x 58 mm

Commit message: Add files via upload
Connections:
- C6 pad 1: +12V -> +BATT
- U8 pad 1: +12V -> +BATT
Routing:
- net +BATT: track 12.8 -> 48.9 mm
- net +12V: track 173.8 -> 142.6 mm
- net /Vsys: track 93.5 -> 94.8 mm

Commit message: Add files via upload
Parts:
- removed C11, C12: 0.1uF, Capacitor_SMD:C_0805_2012Metric
- removed U6, U7: OPA2277, Package_SO:SOIC-8_3.9x4.9mm_P1.27mm
- U4, U5: value OPA2277 -> LT1469
- moved C2 12.4 mm to (103.4, 95.5)
- moved U5 7.96 mm to (98.3, 104.3), turned to 0 degrees
- moved C10 7.84 mm to (98.4, 104.1), turned to 0 degrees
- moved C4 5.66 mm to (96.7, 110.1), turned to 90 degrees
- moved C9 3.30 mm to (98.2, 92.9), turned to 0 degrees
- moved U4 3.07 mm to (98.3, 92.9), turned to 0 degrees
- moved C1 1.87 mm to (91.7, 91.4), turned to 90 degrees
- moved C3 0.16 mm to (91.1, 103.5)
Connections:
- C4 pad 1: Net-(U1-I_{OUT}B) -> /Ch2
- C4 pad 2: /Ch2 -> Net-(U1-I_{OUT}B)
- U1 pad 13: Net-(U1-V_{REF}B) -> Vref
- U1 pad 14: Net-(U1-R_{COM}B) -> Vref
- U1 pad 17: Vref -> /Ch2
- U1 pad 3: Vref -> /Ch1
- U1 pad 6: Net-(U1-R_{COM}A) -> Vref
- U1 pad 7: Net-(U1-V_{REF}A) -> Vref
- U2 pad 13: Net-(U2-V_{REF}B) -> Vref
- U2 pad 14: Net-(U2-R_{COM}B) -> Vref
- U2 pad 17: Vref -> /Ch4
- U2 pad 3: Vref -> /Ch3
- U2 pad 6: Net-(U2-R_{COM}A) -> Vref
- U2 pad 7: Net-(U2-V_{REF}A) -> Vref
- U4 pad 1: Net-(U2-V_{REF}A) -> /Ch3
- U4 pad 2: Net-(U2-R_{COM}A) -> Net-(U2-I_{OUT}A)
- U4 pad 6: Net-(U2-I_{OUT}A) -> Net-(U2-I_{OUT}B)
- U4 pad 7: /Ch3 -> /Ch4
- U5 pad 1: Net-(U2-V_{REF}B) -> /Ch1
- U5 pad 2: Net-(U2-R_{COM}B) -> Net-(U1-I_{OUT}A)
- U5 pad 6: Net-(U2-I_{OUT}B) -> Net-(U1-I_{OUT}B)
- U5 pad 7: /Ch4 -> /Ch2
Routing:
- net +12V: track 142.6 -> 127.0 mm, vias 5 -> 4
- net -12V: track 126.7 -> 114.9 mm, vias 4 -> 3
- net Net-(U1-V_{REF}B): track 11.0 -> 0.00 mm
- net Net-(U2-V_{REF}B): track 10.8 -> 0.00 mm
- net /Ch2: track 23.8 -> 34.1 mm
- net Net-(U2-I_{OUT}B): track 16.2 -> 6.24 mm
- net GND: track 13.2 -> 22.1 mm, vias 19 -> 18
- net Net-(U1-R_{COM}B): track 6.84 -> 0.00 mm
- net Net-(U2-R_{COM}B): track 6.76 -> 0.00 mm
- net Net-(U2-R_{COM}A): track 6.55 -> 0.00 mm
- net Net-(U1-R_{COM}A): track 6.44 -> 0.00 mm
- net Net-(U2-V_{REF}A): track 6.23 -> 0.00 mm
- net Net-(U1-V_{REF}A): track 6.12 -> 0.00 mm
- net Net-(U2-I_{OUT}A): track 22.4 -> 17.1 mm, vias 2 -> 0
- net /Ch4: track 23.2 -> 27.7 mm
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