File: programs/DAC8822/pcb/DAC8822.kicad_sch (KiCad schematic)
At the start: 17 parts, among them J1 TFT ST7735, U1 8BVG4, U2 8BVG4, U3 RP2350B-WeAct, U4 OPA2277, U5 OPA2277, U6 OPA2277, U7 OPA2277, U8 LM7805

Commit message: Add files via upload
Parts:
- added J2, J3, J5, J6: Conn_01x04_Pin, Connector_PinHeader_1.00mm:PinHeader_1x04_P1.00mm_Vertical, symbol Connector:Conn_01x04_Pin
- added J4: Screw_Terminal_01x02, TerminalBlock:TerminalBlock_Xinya_XY308-2.54-2P_1x02_P2.54mm_Horizontal, symbol Connector:Screw_Terminal_01x02
Connections:
- net +10V is gone; now on net Vref: U2.3 (R_{OFS}A), U2.5 (R_{1}A)
- net Ch1: now also J3.1 (Pin_1)
- net Ch2: now also J3.4 (Pin_4)
- net Ch3: now also J2.1 (Pin_1)
- net Ch4: now also J2.4 (Pin_4)
- net GND: now also J2.2 (Pin_2), J2.3 (Pin_3), J3.2 (Pin_2), J3.3 (Pin_3), J4.1 (Pin_1), J6.4 (Pin_4)
- net Vref: now also U2.15 (R_{1}B), U2.17 (R_{OFS}B)
- net +BATT: now reaches U9.1 (VIN)
- net +BATT: now also J4.2 (Pin_2)
- net Btn1: now reaches U3.38 (GPIO32)
- net Btn1: now also J5.1 (Pin_1)
- net Btn2: now reaches U3.39 (GPIO33)
- net Btn2: now also J5.2 (Pin_2)
- net Btn3: now reaches U3.40 (GPIO34)
- net Btn3: now also J5.3 (Pin_3)
- net Btn4: now reaches U3.41 (GPIO35)
- net Btn4: now also J5.4 (Pin_4)
- net Pot1: now reaches U3.46 (GPIO40_ADC0)
- net Pot1: now also J6.2 (Pin_2)
- net Pot2: now reaches U3.47 (GPIO41_ADC1)
- net Pot2: now also J6.3 (Pin_3)
- net +3.3V: now reaches U3.55 (3V3)
- net +3.3V: now also U3.56 (3V3), J6.1 (Pin_1)
- no-connect marks 0 -> 18
Other:
- moved on the sheet: C1, C2, C3, C4, D1, J1, U1, U2, U3, U4A, U4B, U5A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

Commit message: Add files via upload
Parts:
- added R1: 100, Resistor_SMD:R_0805_2012Metric, symbol Device:R
- added R2: 3k, Resistor_SMD:R_0805_2012Metric, symbol Device:R
- added R3: 1k, Resistor_SMD:R_0805_2012Metric, symbol Device:R
- added U10: TL431LP, Package_TO_SOT_THT:TO-92_Inline, symbol Reference_Voltage:TL431LP
Connections:
- net +12V: now also R1.1
- net +5V: no longer J1.1 (Pin_1)
- net GND: now also R3.2, U10.2 (A)
- net Vref: now also R1.2, R2.1, U10.3 (K)
- net VSYS renamed Vsys
- net Vsys: now also J1.1 (Pin_1)
- new net: R2.2, R3.1, U10.1 (REF)
Other:
- company: (none) -> Marc Pelletier
- title: (none) -> 4 Ch Signal Generato Pico 2350 and DAC8822 x 2
- moved on the sheet: C1, C2, C3, C4, C5, C6, J1, J2, J3, U1, U2, U4A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

Commit message: Add files via upload
Parts:
- J2, J3, J5, J6: footprint Connector_PinHeader_1.00mm:PinHeader_1x04_P1.00mm_Vertical -> Connector_PinHeader_1.27mm:PinHeader_1x04_P1.27mm_Vertical
Connections:
- net Vref: now also R2.2; no longer R2.1
- net at R3.1, U10.1 (REF): now also R2.1; no longer R2.2
Other:
- moved on the sheet: R2
Changed lines of the file:
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@@
 	)
 	(junction
-		(at 142.24 182.88)
-		(diameter 0)
-		(color 0 0 0 0)
-	)
-	(junction
-		(at 142.24 175.26)
-		(diameter 0)
-		(color 0 0 0 0)
-	)
-	(junction
 		(at 60.96 35.56)
 		(diameter 0)
@@
 	)
 	(junction
+		(at 142.24 175.26)
+		(diameter 0)
+		(color 0 0 0 0)
+	)
+	(junction
 		(at 88.9 176.53)
 		(diameter 0)
@@
 	)
 	(junction
+		(at 142.24 182.88)
+		(diameter 0)
+		(color 0 0 0 0)
+	)
+	(junction
 		(at 59.69 115.57)
 		(diameter 0)
@@
 	(wire
 		(pts
-			(xy 142.24 175.26) (xy 148.59 175.26)
-		)
-		(stroke
-			(width 0)
-			(type default)
-		)
-	)
-	(wire
-		(pts
 			(xy 110.49 176.53) (xy 113.03 176.53)
 		)
@@
 	(wire
 		(pts
+			(xy 142.24 175.26) (xy 148.59 175.26)
+		)
+		(stroke
+			(width 0)
+			(type default)
+		)
+	)
+	(wire
+		(pts
 			(xy 116.84 67.31) (xy 120.65 67.31)
 		)
@@
 			)
 		)
-		(property "Footprint" "Connector_PinHeader_1.00mm:PinHeader_1x04_P1.00mm_Vertical"
+		(property "Footprint" "Connector_PinHeader_1.27mm:PinHeader_1x04_P1.27mm_Vertical"
 			(at 222.25 67.31 0)
 			(effects
@@
 		)
 		(property "Value" "GND"
-			(at 219.202 96.012 0)
+			(at 214.122 95.504 0)
 			(effects
 				(font
@@
 			)
 		)
-		(property "Footprint" "Connector_PinHeader_1.00mm:PinHeader_1x04_P1.00mm_Vertical"
+		(property "Footprint" "Connector_PinHeader_1.27mm:PinHeader_1x04_P1.27mm_Vertical"
 			(at 45.72 49.53 0)
 			(effects
@@
 	(symbol
 		(lib_id "Device:R")
-		(at 142.24 179.07 0)
+		(at 142.24 179.07 180)
 		(unit 1)
 		(exclude_from_sim no)
@@
 		(dnp no)
 		(property "Reference" "R2"
-			(at 144.018 178.054 0)
+			(at 140.462 180.086 0)
 			(effects
 				(font
@@
 		)
 		(property "Value" "3k"
-			(at 144.018 180.594 0)
+			(at 140.462 177.546 0)
 			(effects
 				(font
@@
 		)
 		(property "Footprint" "Resistor_SMD:R_0805_2012Metric"
-			(at 140.462 179.07 90)
+			(at 144.018 179.07 90)
 			(effects
 				(font
@@
 		(on_board yes)
 		(dnp no)
-		(fields_autoplaced yes)
 		(property "Reference" "#PWR040"
 			(at 217.17 88.9 0)
@@
 		)
 		(property "Value" "+3.3V"
-			(at 217.17 80.01 0)
+			(at 215.138 81.788 0)
 			(effects
 				(font
@@
 			)
 		)
-		(property "Footprint" "Connector_PinHeader_1.00mm:PinHeader_1x04_P1.00mm_Vertical"
+		(property "Footprint" "Connector_PinHeader_1.27mm:PinHeader_1x04_P1.27mm_Vertical"
 			(at 45.72 113.03 0)
 			(effects
@@
 			)
 		)
-		(property "Footprint" "Connector_PinHeader_1.00mm:PinHeader_1x04_P1.00mm_Vertical"
+		(property "Footprint" "Connector_PinHeader_1.27mm:PinHeader_1x04_P1.27mm_Vertical"
 			(at 222.25 87.63 0)
 			(effects

Commit message: Add files via upload
Parts:
- added C10, C11, C12, C7, C8, C9: 0.1uF, Capacitor_SMD:C_0805_2012Metric, symbol Device:C_Small
Connections:
- net +12V: now also C10.2, C11.2, C12.2, C9.2
- net +5V: now also C7.2, C8.2
- net -12V: now also C10.1, C11.1, C12.1, C9.1
- net GND: now also C7.1, C8.1
- net Adj: now reaches R2.1, R3.1, U10.1 (REF)
Other:
- moved on the sheet: C1, C2, C3, C4, C5, C6, D1, J1, J2, J3, J4, J5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

Commit message: Add files via upload
Connections:
- net +12V: no longer C6.1, U8.1 (VI)
- net +BATT: now also C6.1, U8.1 (VI)
Other:
- title: 4 Ch Signal Generato Pico 2350 and DAC8822 x 2 -> 4 Ch Signal Generator Pico 2350 and DAC8822 x 2
- moved on the sheet: C10, C11, C12, C5, C6, C9, J4, R1, R2, R3, U10, U4C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

Commit message: Add files via upload
Parts:
- removed C11, C12: 0.1uF, Capacitor_SMD:C_0805_2012Metric, symbol Device:C_Small
- removed U6, U7: OPA2277, Package_SO:SOIC-8_3.9x4.9mm_P1.27mm, symbol Amplifier_Operational:OPA2277
Connections:
- net Ch1: now also U1.3 (R_{OFS}A), U5.1
- net Ch2: now also C4.1, U1.17 (R_{OFS}B), U5.7; no longer C4.2
- net Ch3: now also U2.3 (R_{OFS}A), U4.1; no longer U4.7
- net Ch4: now also U2.17 (R_{OFS}B), U4.7; no longer U5.7
- net Vref: now also U1.13 (V_{REF}B), U1.14 (R_{COM}B), U1.6 (R_{COM}A), U1.7 (V_{REF}A), U2.13 (V_{REF}B), U2.14 (R_{COM}B), U2.6 (R_{COM}A), U2.7 (V_{REF}A); no longer U1.17 (R_{OFS}B), U1.3 (R_{OFS}A), U2.17 (R_{OFS}B), U2.3 (R_{OFS}A)
- net at C2.1, U2.12 (I_{OUT}B): now also U4.6 (-); no longer U5.6 (-)
- net at U5.2 (-): now also C3.1, U1.8 (I_{OUT}A); no longer U2.14 (R_{COM}B)
- net at U4.2 (-): now also C1.1, U2.8 (I_{OUT}A); no longer U2.6 (R_{COM}A)
- net at U1.12 (I_{OUT}B): now also C4.2, U5.6 (-); no longer C4.1
Other:
- moved on the sheet: C1, C10, C2, C4, C7, C8, C9, J2, J3, U4C, U5C
